File: hardware/relay.kicad_sch (KiCad schematic)
At the start: 4 parts, among them K1 G5Q-1, U2 TCMT1100

Commit message: chore(hw): migrate KiCad files to the KiCad 10 format
Via `kicad-cli sch upgrade` / `pcb upgrade` (bread-infra
scripts/upgrade_kicad10.sh). Verified lossless: identical netlist, footprint
positions and routing.

Note `sch upgrade` does not cascade into hierarchical sub-sheets, so every
.kicad_sch is upgraded individually -- upgrading only the root sheet leaves
sub-sheets on the old format, which looks migrated and is not.
Parts:
- renumbered D6 to D8, K1 to K3, R1 to R3, U2 to U4
