File: hardware/BREAD_Slice.kicad_pcb (KiCad board)
At the start: 2 copper layers, 70 x 100 mm, 45 parts, among them J1 Conn_01x10_Female, J1 I2C_01x04, J2 Screw_Terminal_01x04, J3 Screw_Terminal_01x03, J4 Screw_Terminal_01x03, J5 Screw_Terminal_01x03, J6 Screw_Terminal_01x03, K1 G5Q-1, K2 G5Q-1, K3 G5Q-1, K4 G5Q-1, U2 TCMT1100, U3 TCMT1100, U4 TCMT1100, U5 TCMT1100

Commit message: fix(hw): re-point stale library nicknames
These parts exist in KiCad-Master-Lib; the boards referenced libraries that no
longer exist (kml-custom, KML-Custom, and SparkFun libraries that never
contained the part) or names the library has since changed.

KiCad embeds footprint geometry in the .kicad_pcb, so the boards rendered and
fabricated correctly and the rot stayed invisible -- it only surfaces on
update-from-library, or when a generator tries to resolve a nickname.

Nickname/name only. No geometry is changed:

  KMLib_Mounting:Thermal Pad -> KMLib_Mounting:Thermal_Pad

Only references that failed to resolve were touched. Generic parts (<=4 pins)
and KiCad *-rescue libraries are deliberately excluded: fingerprint matching
cannot distinguish a 2-pin resistor from a 2-pin capacitor, so those are being
done by hand.
Parts:
- HS1: footprint KMLib_Mounting:Thermal Pad -> KMLib_Mounting:Thermal_Pad
Changed lines of the file:
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@@
 		(embedded_fonts no)
 	)
-	(footprint "KMLib_Mounting:Thermal Pad"
+	(footprint "KMLib_Mounting:Thermal_Pad"
 		(layer "F.Cu")
 		(at 131.35 121.355)
